Commit message: Added dual arm moveit configurations (left, right)

File: franka_description/robots/dual_panda_arm.urdf.xacro (robot description, xacro)
@@ -9,7 +9,21 @@
   <xacro:arg name="use_fake_hardware" default="false"/>
   <xacro:arg name="fake_sensor_commands" default="false"/>
+  <link name="base_link">
+    <visual>
+      <geometry>
+         <box size="0.1 0.1 0.1"/>
+      </geometry>
+      <origin rpy="0 0 0" xyz="0 0 0"/>
+    </visual>
+    <collision>
+      <geometry>
+         <box size="0.1 0.1 0.1"/>
+      </geometry>
+      <origin rpy="0 0 0" xyz="0 0 0"/>
+    </collision>
+  </link>
   <xacro:include filename="$(find franka_description)/robots/panda_arm.xacro"/>
-  <xacro:panda_arm arm_id="$(arg arm_id_1)" connected_to="base_link" rpy="${-90 * pi/180} 0 ${-90 * pi/180}"  xyz="-143.26e-3 +200e-3 924.51e-3" safety_distance="0.03"/>
-  <xacro:panda_arm arm_id="$(arg arm_id_2)" connected_to="base_link" rpy="${+90 * pi/180} 0 ${+90 * pi/180}"  xyz="-143.26e-3 -200e-3 924.51e-3" safety_distance="0.03"/>
+  <xacro:panda_arm arm_id="$(arg arm_id_1)" connected_to="base_link" rpy="${-90 * pi/180} 0 ${-90 * pi/180}"  xyz="-143.26e-3 +600e-3 924.51e-3" safety_distance="0.03"/>
+  <xacro:panda_arm arm_id="$(arg arm_id_2)" connected_to="base_link" rpy="${+90 * pi/180} 0 ${+90 * pi/180}"  xyz="-143.26e-3 -600e-3 924.51e-3" safety_distance="0.03"/>
   <xacro:if value="$(arg hand_1)">
     <xacro:include filename="$(find franka_description)/robots/hand.xacro"/>
@@ -22,18 +36,3 @@
   <xacro:include filename="$(find franka_description)/robots/dual_panda_arm.ros2_control.xacro"/>
   <xacro:panda_arm_ros2_control ns_1="$(arg arm_id_1)" ns_2="$(arg arm_id_2)" robot_ip_1="$(arg robot_ip_1)" robot_ip_2="$(arg robot_ip_2)" use_fake_hardware="$(arg use_fake_hardware)" fake_sensor_commands="$(arg fake_sensor_commands)"/>
-  <link name="base_link">
-    <visual>
-      <geometry>
-         <box size="0.20 0.23 0.26"/>
-      </geometry>
-      <origin rpy="0 0 0" xyz="0 0 0.1"/>
-    </visual>
-    <collision>
-      <geometry>
-         <box size="0.20 0.23 0.26"/>
-        <cylinder length="0.23" radius="0.09"/>
-      </geometry>
-      <origin rpy="0 0 0" xyz="0 0 0.1"/>
-    </collision>
-  </link>
 </robot>
