Commit message: icra24 expo version

File: franka_description/robots/dual_panda_arm_sim.ros2_control.xacro (robot description, xacro)
@@ -1,18 +1,15 @@
 <?xml version="1.0"?>
 <robot xmlns:xacro="http://www.ros.org/wiki/xacro">
-  <xacro:macro name="panda_arm_ros2_control" params="ns_1 robot_ip_1 use_fake_hardware:=^|false fake_sensor_commands:=^|false">
-    <ros2_control name="FrankaMultiHardwareInterface" type="system">
+  <xacro:macro name="panda_arm_sim_ros2_control" params="ns_1 ns_2 hand_1 hand_2 scene_xml mj_yaml">
+    <ros2_control name="FrankaMujocoMultiHardwareInterface" type="system">
       <hardware>
-        <param name="robot_count">1</param>
-        <xacro:if value="${use_fake_hardware}">
-          <plugin>fake_components/GenericSystem</plugin>
-          <param name="fake_sensor_commands">${fake_sensor_commands}</param>
-          <param name="state_following_offset">0.0</param>
-        </xacro:if>
-        <xacro:unless value="${use_fake_hardware}">
-          <plugin>franka_hardware/FrankaMultiHardwareInterface</plugin>
-          <param name="robot_ip_1">${robot_ip_1}</param>
-        </xacro:unless>
+        <param name="robot_count">2</param>
+        <plugin>franka_hardware/FrankaMujocoMultiHardwareInterface</plugin>
         <param name="ns_1">${ns_1}</param>
+        <param name="ns_2">${ns_2}</param>
+        <param name="hand_1">${hand_1}</param>
+        <param name="hand_2">${hand_2}</param>
+        <param name="scene_xml">${scene_xml}</param>
+        <param name="mj_yaml">${mj_yaml}</param>
       </hardware>
       <xacro:macro name="configure_joint" params="joint_name initial_position">
@@ -34,4 +31,11 @@
       <xacro:configure_joint joint_name="${ns_1}_joint6" initial_position="${pi/2}"/>
       <xacro:configure_joint joint_name="${ns_1}_joint7" initial_position="${pi/4}"/>
+      <xacro:configure_joint joint_name="${ns_2}_joint1" initial_position="0.0"/>
+      <xacro:configure_joint joint_name="${ns_2}_joint2" initial_position="${-pi/4}"/>
+      <xacro:configure_joint joint_name="${ns_2}_joint3" initial_position="0.0"/>
+      <xacro:configure_joint joint_name="${ns_2}_joint4" initial_position="${-3*pi/4}"/>
+      <xacro:configure_joint joint_name="${ns_2}_joint5" initial_position="0.0"/>
+      <xacro:configure_joint joint_name="${ns_2}_joint6" initial_position="${pi/2}"/>
+      <xacro:configure_joint joint_name="${ns_2}_joint7" initial_position="${pi/4}"/>
     </ros2_control>
   </xacro:macro>

File: franka_description/robots/panda_arm.ros2_control.xacro (robot description, xacro)
@@ -2,6 +2,7 @@
 <robot xmlns:xacro="http://www.ros.org/wiki/xacro">
   <xacro:macro name="panda_arm_ros2_control" params="ns robot_ip use_fake_hardware:=^|false fake_sensor_commands:=^|false">
-    <ros2_control name="FrankaHardwareInterface" type="system">
+    <ros2_control name="FrankaMultiHardwareInterface" type="system">
       <hardware>
+        <param name="robot_count">1</param>
         <xacro:if value="${use_fake_hardware}">
           <plugin>fake_components/GenericSystem</plugin>
@@ -10,7 +11,8 @@
         </xacro:if>
         <xacro:unless value="${use_fake_hardware}">
-          <plugin>franka_hardware/FrankaHardwareInterface</plugin>
-          <param name="robot_ip">${robot_ip}</param>
+          <plugin>franka_hardware/FrankaMultiHardwareInterface</plugin>
+          <param name="robot_ip_1">${robot_ip}</param>
         </xacro:unless>
+        <param name="ns_1">${ns}</param>
       </hardware>
       <xacro:macro name="configure_joint" params="joint_name initial_position">

File: franka_description/robots/panda_arm_sim.ros2_control.xacro (robot description, xacro)
@@ -1,11 +1,13 @@
 <?xml version="1.0"?>
 <robot xmlns:xacro="http://www.ros.org/wiki/xacro">
-  <xacro:macro name="panda_arm_sim_ros2_control" params="ns hand scene_xml">
+  <xacro:macro name="panda_arm_sim_ros2_control" params="ns hand scene_xml mj_yaml">
     <ros2_control name="FrankaMujocoHardwareInterface" type="system">
       <hardware>
-        <plugin>franka_hardware/FrankaMujocoHardwareInterface</plugin>
-        <param name="ns">${ns}</param>
-        <param name="hand">${hand}</param>
+        <param name="robot_count">1</param>
+        <plugin>franka_hardware/FrankaMujocoMultiHardwareInterface</plugin>
+        <param name="ns_1">${ns}</param>
+        <param name="hand_1">${hand}</param>
         <param name="scene_xml">${scene_xml}</param>
+        <param name="mj_yaml">${mj_yaml}</param>
       </hardware>
       <xacro:macro name="configure_joint" params="joint_name initial_position">
@@ -13,4 +15,5 @@
           <param name="initial_position">${initial_position}</param>
           <command_interface name="effort"/>
+          <command_interface name="position"/>
           <command_interface name="velocity"/>
           <state_interface name="effort"/>

File: franka_description/robots/panda_arm_sim.urdf.xacro (robot description, xacro)
@@ -4,4 +4,5 @@
   <xacro:arg name="hand" default="true"/> <!-- Should a franka_gripper be mounted at the flange?" -->
   <xacro:arg name="scene_xml" default="scene.xml"/> <!-- Path to the scene_xml -->
+  <xacro:arg name="mj_yaml" default=""/> <!-- Path to the scene_xml -->
   <xacro:include filename="$(find franka_description)/robots/panda_arm.xacro"/>
   <xacro:panda_arm arm_id="$(arg arm_id)" safety_distance="0.03"/>
@@ -11,4 +12,4 @@
   </xacro:if>
   <xacro:include filename="$(find franka_description)/robots/panda_arm_sim.ros2_control.xacro"/>
-  <xacro:panda_arm_sim_ros2_control ns="$(arg arm_id)" hand="$(arg hand)" scene_xml="$(arg scene_xml)"/>
+  <xacro:panda_arm_sim_ros2_control ns="$(arg arm_id)" hand="$(arg hand)" scene_xml="$(arg scene_xml)" mj_yaml="$(arg mj_yaml)"/>
 </robot>
