Commit message: moved virtual joint to the parent moveit xacro file

File: franka_moveit_config/srdf/dual_panda_arm.srdf.xacro (robot description, xacro)
@@ -3,13 +3,13 @@
   <xacro:arg name="arm_id_1" default="left"/>
   <xacro:arg name="arm_id_2" default="right"/>
-  <xacro:arg name="parent_frame" default="world"/>
   <xacro:arg name="hand_1" default="false"/>
   <xacro:arg name="hand_2" default="false"/>
+  <xacro:arg name="parent_frame" default="world"/>
   <xacro:property name="arm_id_1" value="$(arg arm_id_1)"/>
   <xacro:property name="arm_id_2" value="$(arg arm_id_2)"/>
-  <xacro:property name="parent_frame" value="$(arg parent_frame)"/>
   <xacro:include filename="$(find franka_moveit_config)/srdf/multi_panda_arm.xacro"/>
-  <xacro:panda_arm arm_id="${arm_id_1}" parent_frame="${parent_frame}"/>
-  <xacro:panda_arm arm_id="${arm_id_2}" parent_frame="${parent_frame}"/>
+  <xacro:panda_arm arm_id="${arm_id_1}" />
+  <xacro:panda_arm arm_id="${arm_id_2}" />
+  <virtual_joint name="virtual_joint" type="fixed" parent_frame="$(arg parent_frame)" child_link="base_link"/>
   <group name="dual_panda_arm">
     <group name="${arm_id_1}_arm" />

File: franka_moveit_config/srdf/multi_panda_arm.xacro (robot description, xacro)
@@ -1,9 +1,8 @@
 <?xml version="1.0" ?>
 <robot xmlns:xacro="http://www.ros.org/wiki/xacro" name="panda">
-  <xacro:macro name="panda_arm" params="arm_id:='panda' parent_frame:='world' ">
+  <xacro:macro name="panda_arm" params="arm_id:='panda'">
     <xacro:include filename="$(find franka_moveit_config)/srdf/group_definition.xacro"/>
     <xacro:group_definition arm_id="${arm_id}" group_name="${arm_id}_manipulator" tip_link="${arm_id}_hand_tcp"/>
     <xacro:group_definition arm_id="${arm_id}" group_name="${arm_id}_arm" tip_link="${arm_id}_link8"/>
-    <virtual_joint name="virtual_joint" type="fixed" parent_frame="${parent_frame}" child_link="${arm_id}_link0"/>
     <disable_collisions link1="${arm_id}_link0" link2="${arm_id}_link1" reason="Adjacent"/>
     <disable_collisions link1="${arm_id}_link0" link2="${arm_id}_link2" reason="Never"/>
